File: Hardware/PCB/LED_Coaster.kicad_pcb (KiCad board)
At the start: 2 copper layers, 90 x 90 mm, 55 parts, among them J1 Input voltage, J2 Boot Option, J3 JTAG, J4 UART, SW1 SW_SPST, SW2 SW_DIP_x01, SW3 SW_DIP_x01, U1 ESP32-C3-WROOM-02-H4, U2 MCP1792x-3302xDB

Commit message: Latest and gratest PCB files from boa himself
Parts:
- removed H2: MountingHole, MountingHole:MountingHole_4.3mm_M4_Pad_Via
- removed J2: Boot Option, Connector_PinHeader_2.54mm:PinHeader_1x02_P2.54mm_Vertical
- removed SW2, SW3: SW_DIP_x01, Button_Switch_SMD:SW_SPDT_PCM12
- removed U2: MCP1792x-3302xDB, Package_TO_SOT_SMD:SOT-223-3_TabPin2
- added Btn1: button, Button_Switch_SMD:SW_SPST_SKQG_WithStem, F.Cu at (187.6, 94.6)
- added Btn2: button, Button_Switch_SMD:SW_SPST_SKQG_WithStem, F.Cu at (182.4, 103.1)
- added Btn3: Boot, Button_Switch_SMD:SW_SPST_SKQG_WithStem, F.Cu at (162.9, 40.4)
- added C6: 4.7uF, Capacitor_SMD:C_0805_2012Metric_Pad1.18x1.45mm_HandSolder, F.Cu at (140.2, 45.9)
- added C7: 4.7uF, Capacitor_SMD:C_0805_2012Metric_Pad1.18x1.45mm_HandSolder, F.Cu at (145.4, 50.6)
- added D33: LED, LED_SMD:LED_0805_2012Metric_Pad1.15x1.40mm_HandSolder, F.Cu at (150.3, 79.8)
- added D34: LED, LED_SMD:LED_0805_2012Metric_Pad1.15x1.40mm_HandSolder, F.Cu at (184.5, 61.7)
- added R10: 22, Resistor_SMD:R_0805_2012Metric_Pad1.20x1.40mm_HandSolder, F.Cu at (176.5, 91.8)
- added R11: 22, Resistor_SMD:R_0805_2012Metric_Pad1.20x1.40mm_HandSolder, F.Cu at (178.7, 91.8)
- added R12: 1k, Resistor_SMD:R_0805_2012Metric_Pad1.20x1.40mm_HandSolder, F.Cu at (184.5, 59.3)
- added R2: 2k, Resistor_SMD:R_0805_2012Metric_Pad1.20x1.40mm_HandSolder, F.Cu at (137.8, 50.5)
- added R5: 1k, Resistor_SMD:R_0805_2012Metric_Pad1.20x1.40mm_HandSolder, F.Cu at (147.1, 79.8)
- added R6: 5.1K, Resistor_SMD:R_0805_2012Metric_Pad1.20x1.40mm_HandSolder, F.Cu at (154.4, 45.7)
- added R9: 1k, Resistor_SMD:R_0805_2012Metric_Pad1.20x1.40mm_HandSolder, F.Cu at (180.9, 95.1)
- added SW1: SW_SPDT, Button_Switch_SMD:SW_SPDT_CK_JS102011SAQN, F.Cu at (136.3, 38.9)
- added U3: MCP73831-2-OT, Package_TO_SOT_SMD:SOT-23-5, F.Cu at (141.5, 50.5)
- added U4: AMS1117-3.3, Package_TO_SOT_SMD:SOT-223-3_TabPin2, F.Cu at (122.3, 56.6)
- Btn4: renamed from SW1; value SW_SPST -> Enable
- C3, R1, R3, R4, U1: moved to F.Cu
- D1, D10, D11, D12, D13, D14, D15, D16, D17, D18, D19, D2, D20, D21, D22, D23, D24, D25, D26, D27, D28, D29, D3, D30, D4, D5, D6, D7, D8, D9: footprint LED_SMD:LED_WS2812B_PLCC4_5.0x5.0mm_P3.2mm -> Library:LED_WS2812_5050_handsolder
- D31, D32: value LED -> SS34; footprint LED_SMD:LED_0805_2012Metric_Pad1.15x1.40mm_HandSolder -> Diode_SMD:D_SMA
- J1: value Input voltage -> Li-po; footprint Connector_PinHeader_2.54mm:PinHeader_1x02_P2.54mm_Vertical -> Connector_JST:JST_EH_S2B-EH_1x02_P2.50mm_Horizontal; moved to B.Cu
- J3: value JTAG -> USB_C_Receptacle_USB2.0_16P; footprint Connector_PinHeader_2.54mm:PinHeader_1x04_P2.54mm_Vertical -> Connector_USB:USB_C_Receptacle_HRO_TYPE-C-31-M-12
- R7: value 150 -> 5.1K
- R8: value 150 -> 1k
- moved C2 67.5 mm to (189.4, 65.7), turned to -90 degrees
- moved C1 63.9 mm to (186.9, 65.7), turned to 90 degrees
- moved D31 56.6 mm to (131.4, 50.6), turned to 0 degrees
- moved J4 56.4 mm to (154.2, 120.9), turned to -90 degrees
- moved J3 55.3 mm to (149.9, 38.0), turned to 180 degrees
- moved D32 47.8 mm to (131.4, 46.6), turned to 0 degrees
- moved R7 41.2 mm to (145.4, 45.7), turned to -90 degrees
- moved R8 39.8 mm to (183.5, 91.8), turned to 180 degrees
- moved C3 38.9 mm to (179.7, 53.5), turned to 180 degrees
- moved R1 38.4 mm to (179.7, 55.9), turned to 0 degrees
- moved Btn4 34.0 mm to (174.2, 45.9), turned to -36 degrees
- moved U1 32.6 mm to (181.4, 79.0), turned to -90 degrees
- moved R4 32.1 mm to (175.4, 65.6), turned to -90 degrees
- moved J1 30.5 mm to (139.2, 59.1), turned to 90 degrees
- moved R3 29.2 mm to (183.6, 66.8), turned to 180 degrees
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Connections:
- C4 pad 2: +5V -> +BATT
- D1 pad 1: Net-(D1-VDD) -> +BATT
- D10 pad 1: Net-(D1-VDD) -> +BATT
- D11 pad 1: Net-(D1-VDD) -> +BATT
- D12 pad 1: Net-(D1-VDD) -> +BATT
- D13 pad 1: Net-(D1-VDD) -> +BATT
- D14 pad 1: Net-(D1-VDD) -> +BATT
- D15 pad 1: Net-(D1-VDD) -> +BATT
- D16 pad 1: Net-(D1-VDD) -> +BATT
- D17 pad 1: Net-(D1-VDD) -> +BATT
- D18 pad 1: Net-(D1-VDD) -> +BATT
- D19 pad 1: Net-(D1-VDD) -> +BATT
- D2 pad 1: Net-(D1-VDD) -> +BATT
- D20 pad 1: Net-(D1-VDD) -> +BATT
- D21 pad 1: Net-(D21-VDD) -> +BATT
- D22 pad 1: Net-(D21-VDD) -> +BATT
- D23 pad 1: Net-(D21-VDD) -> +BATT
- D24 pad 1: Net-(D21-VDD) -> +BATT
- D25 pad 1: Net-(D21-VDD) -> +BATT
- D26 pad 1: Net-(D21-VDD) -> +BATT
- D27 pad 1: Net-(D21-VDD) -> +BATT
- D28 pad 1: Net-(D21-VDD) -> +BATT
- D29 pad 1: Net-(D21-VDD) -> +BATT
- D3 pad 1: Net-(D1-VDD) -> +BATT
- D30 pad 1: Net-(D21-VDD) -> +BATT
- D31 pad 1: GND -> Net-(D31-K)
- D32 pad 1: GND -> Net-(D31-K)
- D32 pad 2: Net-(D32-A) -> +5V
- D4 pad 1: Net-(D1-VDD) -> +BATT
- D5 pad 1: Net-(D1-VDD) -> +BATT
- D6 pad 1: Net-(D1-VDD) -> +BATT
- D7 pad 1: Net-(D1-VDD) -> +BATT
- D8 pad 1: Net-(D1-VDD) -> +BATT
- D9 pad 1: Net-(D1-VDD) -> +BATT
- J1 pad 2: +5V -> Net-(D31-A)
- R7 pad 1: Net-(D31-A) -> Net-(J3-CC2)
- R7 pad 2: Net-(D1-VDD) -> GND
- R8 pad 1: Net-(D32-A) -> +3V3
- R8 pad 2: Net-(D21-VDD) -> Net-(Btn1-B)
- U1 pad 13: unconnected-(U1-IO18-Pad13) -> Net-(U1-IO18)
- U1 pad 14: unconnected-(U1-IO19-Pad14) -> Net-(U1-IO19)
- U1 pad 15: unconnected-(U1-IO3-Pad15) -> Net-(Btn2-B)
- U1 pad 16: unconnected-(U1-IO2-Pad16) -> Net-(Btn1-B)
- U1 pad 3: Net-(J3-Pin_1) -> unconnected-(U1-IO4-Pad3)
- U1 pad 4: Net-(J3-Pin_2) -> unconnected-(U1-IO5-Pad4)
- U1 pad 5: Net-(J3-Pin_3) -> unconnected-(U1-IO6-Pad5)
- U1 pad 6: Net-(J3-Pin_4) -> Net-(D34-A)
Routing:
- net +BATT: track 0.00 -> 318.8 mm, vias 0 -> 2
- net Net-(D1-VDD): track 220.4 -> 0.00 mm, vias 1 -> 0
- net Net-(D21-VDD): track 135.4 -> 0.00 mm, vias 4 -> 0
- net D+: track 0.00 -> 82.8 mm, vias 0 -> 4
- net D-: track 0.00 -> 81.2 mm, vias 0 -> 2
- net Net-(J3-Pin_1): track 71.8 -> 0.00 mm, vias 1 -> 0
- net Net-(J3-Pin_2): track 67.7 -> 0.00 mm, vias 3 -> 0
- net Net-(J3-Pin_3): track 58.3 -> 0.00 mm, vias 4 -> 0
- net /large_ring: track 49.8 -> 7.40 mm, vias 4 -> 1
- net +3V3: track 137.0 -> 95.3 mm, vias 2 -> 5
- net +5V: track 13.7 -> 51.6 mm, vias 0 -> 2
- net Net-(J3-Pin_4): track 35.3 -> 0.00 mm, vias 1 -> 0
- net Net-(Btn3-A): track 63.1 -> 32.8 mm, vias 3 -> 0
- net Net-(U3-STAT): track 0.00 -> 29.8 mm, vias 0 -> 2
- net Net-(D31-A): track 3.40 -> 21.4 mm
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- added copper zone on F.Cu, net +3V3
- added copper zone on F.Cu, net +5V
- added copper zone on F.Cu, net GND
Other:
- outline, holes or cut-outs redrawn
- board text added: "Boot"
- board text added: "Enable"
- board text added: "ON/OFF"
- board text removed: "Inner"
- board text removed: "Outer"
