File: Hardware/PCB/LED_Coaster.kicad_pcb (KiCad board)
At the start: 2 copper layers, 90 x 90 mm, 88 parts, among them J1 Li-po, J3 USB_C_Receptacle_USB2.0_16P, J4 UART, Q1 AO3401A, SW1 SW_SPDT, U1 ESP32-C3-WROOM-02-H4, U3 MCP73871-2CC, U4 TLV75533PDBVR

Commit message: Enlarge U1's stitching vias so they clear annular and hole-to-hole
The twelve GND vias inside the ESP32 module's land pattern were
0.40 mm pads on a 0.30 mm drill: 0.05 mm of annular ring against a
0.13 mm rule, and 0.478 mm hole-to-hole on the 0.778 mm diagonal
against a 0.4995 mm rule. That is 28 of the 139 DRC violations, none
of them from anything drawn on this board.

They are now 0.55 mm pads on a 0.25 mm drill, which gives 0.15 mm of
annular ring and 0.528 mm hole-to-hole. Nothing else moves: the
nearest foreign pad is 0.978 mm away and the nearest other hole is the
next via in the array.

This needs Minimum through hole set to 0.20 mm, which the phase 6 note
now spells out. U3's QFN thermal vias are 0.20 mm and already needed
it; leaving the rule at 0.30 would just swap 16 hole-to-hole errors
for 12 drill errors.

Co-Authored-By: Claude Opus 5 <noreply@anthropic.com>
Routing:
- net GND: track 80.2 -> 86.4 mm, vias 23 -> 30
Changed lines of the file:
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@@
 	(footprint "ESP32-C3-WROOM-02-H4:MODULE_ESP32-C3-WROOM-02-H4"
 		(layer "F.Cu")
-		(at 181.44 79.02 -90)
+		(at 181.44 78.980001 -90)
 		(property "Reference" "U1"
 			(at 0.050001 0.43 90)
@@
 		(pad "28" thru_hole circle
 			(at 0.410001 2.2 270)
-			(size 0.4 0.4)
-			(drill 0.3)
+			(size 0.55 0.55)
+			(drill 0.25)
 			(layers "*.Cu")
 			(remove_unused_layers no)
@@
 		(pad "29" thru_hole circle
 			(at 1.509999 2.2 270)
-			(size 0.4 0.4)
-			(drill 0.3)
+			(size 0.55 0.55)
+			(drill 0.25)
 			(layers "*.Cu")
 			(remove_unused_layers no)
@@
 		(pad "30" thru_hole circle
 			(at -0.14 2.75 270)
-			(size 0.4 0.4)
-			(drill 0.3)
+			(size 0.55 0.55)
+			(drill 0.25)
 			(layers "*.Cu")
 			(remove_unused_layers no)
@@
 		(pad "31" thru_hole circle
 			(at 0.96 2.75 270)
-			(size 0.4 0.4)
-			(drill 0.3)
+			(size 0.55 0.55)
+			(drill 0.25)
 			(layers "*.Cu")
 			(remove_unused_layers no)
@@
 		(pad "32" thru_hole circle
 			(at 2.059998 2.749998 270)
-			(size 0.4 0.4)
-			(drill 0.3)
+			(size 0.55 0.55)
+			(drill 0.25)
 			(layers "*.Cu")
 			(remove_unused_layers no)
@@
 		(pad "33" thru_hole circle
 			(at 0.409997 3.300002 270)
-			(size 0.4 0.4)
-			(drill 0.3)
+			(size 0.55 0.55)
+			(drill 0.25)
 			(layers "*.Cu")
 			(remove_unused_layers no)
@@
 		(pad "34" thru_hole circle
 			(at 1.51 3.3 270)
-			(size 0.4 0.4)
-			(drill 0.3)
+			(size 0.55 0.55)
+			(drill 0.25)
 			(layers "*.Cu")
 			(remove_unused_layers no)
@@
 		(pad "35" thru_hole circle
 			(at -0.140001 3.850002 270)
-			(size 0.4 0.4)
-			(drill 0.3)
+			(size 0.55 0.55)
+			(drill 0.25)
 			(layers "*.Cu")
 			(remove_unused_layers no)
@@
 		(pad "36" thru_hole circle
 			(at 0.960001 3.85 270)
-			(size 0.4 0.4)
-			(drill 0.3)
+			(size 0.55 0.55)
+			(drill 0.25)
 			(layers "*.Cu")
 			(remove_unused_layers no)
@@
 		(pad "37" thru_hole circle
 			(at 2.06 3.85 270)
-			(size 0.4 0.4)
-			(drill 0.3)
+			(size 0.55 0.55)
+			(drill 0.25)
 			(layers "*.Cu")
 			(remove_unused_layers no)
@@
 		(pad "38" thru_hole circle
 			(at 0.41 4.400001 270)
-			(size 0.4 0.4)
-			(drill 0.3)
+			(size 0.55 0.55)
+			(drill 0.25)
 			(layers "*.Cu")
 			(remove_unused_layers no)
@@
 		(pad "39" thru_hole circle
 			(at 1.510004 4.400001 270)
-			(size 0.4 0.4)
-			(drill 0.3)
+			(size 0.55 0.55)
+			(drill 0.25)
 			(layers "*.Cu")
 			(remove_unused_layers no)
@@
 			(polygon
 				(pts
-					(xy 191.440002 70.02) (xy 191.440001 88.020001) (xy 185.439999 88.020001) (xy 185.439999 70.019999)
+					(xy 191.440002 69.980001) (xy 191.440001 87.980002) (xy 185.439999 87.980002) (xy 185.439999 69.98)
 				)
 			)
@@
 			(polygon
 				(pts
-					(xy 191.440002 70.02) (xy 191.440001 88.020001) (xy 185.439999 88.020001) (xy 185.439999 70.019999)
+					(xy 191.440002 69.980001) (xy 191.440001 87.980002) (xy 185.439999 87.980002) (xy 185.439999 69.98)
 				)
 			)
@@
 			(polygon
 				(pts
-					(xy 191.440002 70.02) (xy 191.440001 88.020001) (xy 185.439999 88.020001) (xy 185.439999 70.019999)
+					(xy 191.440002 69.980001) (xy 191.440001 87.980002) (xy 185.439999 87.980002) (xy 185.439999 69.98)
 				)
 			)
@@
 	)
 	(segment
+		(start 129.9 54)
+		(end 130.17 53.73)
+		(width 0.25)
+		(layer "F.Cu")
+		(net "GND")
+	)
+	(segment
 		(start 179.24 80.529999)
 		(end 177.040004 80.529999)
@@
 	)
 	(segment
+		(start 125 59.7)
+		(end 125 57.2)
+		(width 0.25)
+		(layer "F.Cu")
+		(net "GND")
+	)
+	(segment
 		(start 178.37625 61.22375)
 		(end 181.17 61.22375)
@@
 	)
 	(segment
+		(start 125 57.2)
+		(end 125 56.9)
+		(width 0.25)
+		(layer "F.Cu")
+		(net "GND")
+	)
+	(segment
 		(start 160.39 105.79)
 		(end 160.61 105.79)
@@
 	)
 	(segment
+		(start 129.0375 48.0975)
+		(end 129.17 48.23)
+		(width 0.25)
+		(layer "F.Cu")
+		(net "GND")
+	)
+	(segment
 		(start 183.545 59.2925)
 		(end 181.8475 59.2925)
@@
 	)
 	(segment
+		(start 180.74 67.8)
+		(end 181.67 68.73)
+		(width 0.25)
+		(layer "F.Cu")
+		(net "GND")
+	)
+	(segment
 		(start 178.690002 81.079998)
 		(end 177.590002 81.079998)
@@
 	)
 	(segment
+		(start 180.6375 67.8)
+		(end 180.74 67.8)
+		(width 0.25)
+		(layer "F.Cu")
+		(net "GND")
+	)
+	(segment
 		(start 172.34 68.94)
 		(end 171.37 67.97)
@@
 	)
 	(segment
+		(start 129.0375 51)
+		(end 129.0375 51.0975)
+		(width 0.25)
+		(layer "F.Cu")
+		(net "GND")
+	)
+	(segment
 		(start 145.42 46.73)
 		(end 147.13 46.73)
@@
 	)
 	(segment
+		(start 129.0375 48)
+		(end 129.0375 48.0975)
+		(width 0.25)
+		(layer "F.Cu")
+		(net "GND")
+	)
+	(segment
 		(start 186.91 64.6925)
 		(end 186.91 63.61)
@@
 	)
 	(segment
+		(start 129.0375 51.0975)
+		(end 129.17 51.23)
+		(width 0.25)
+		(layer "F.Cu")
+		(net "GND")
+	)
+	(segment
 		(start 160.39 105.8)
 		(end 160.39 105.79)
@@
 	)
 	(segment
+		(start 120.5 57.2)
+		(end 120.64 57.2)
+		(width 0.25)
+		(layer "F.Cu")
+		(net "GND")
+	)
+	(segment
 		(start 178.69 78.88)
 		(end 178.69 79.98)
@@
 	)
 	(segment
+		(start 129.0375 54)
+		(end 129.9 54)
+		(width 0.25)
+		(layer "F.Cu")
+		(net "GND")
+	)
+	(segment
 		(start 155.04 46.73)
 		(end 156.09 45.68)
@@
 	)
 	(segment
+		(start 120.64 57.2)
+		(end 120.67 57.23)
+		(width 0.25)
+		(layer "F.Cu")
+		(net "GND")
+	)
+	(segment
 		(start 146.545002 42.075002)
 		(end 145.629999 41.159999)
@@
 	)
 	(via
+		(at 120.67 57.23)
+		(size 0.8)
+		(drill 0.4)
+		(layers "F.Cu" "B.Cu")
+		(net "GND")
+	)
+	(via
+		(at 122.67 108.73)
+		(size 0.8)
+		(drill 0.4)
+		(layers "F.Cu" "B.Cu")
+		(net "GND")
+	)
+	(via
 		(at 171.37 67.97)
 		(size 0.8)
@@
 	)
 	(via
+		(at 125 57.2)
+		(size 0.8)
+		(drill 0.4)
+		(layers "F.Cu" "B.Cu")
+		(net "GND")
+	)
+	(via
 		(at 155.17 63.979999)
 		(size 0.8)
@@
 	)
 	(via
+		(at 181.67 68.73)
+		(size 0.8)
+		(drill 0.4)
+		(layers "F.Cu" "B.Cu")
+		(net "GND")
+	)
+	(via
 		(at 170.82 41.37)
 		(size 0.8)
@@
 	)
 	(via
+		(at 130.17 53.73)
+		(size 0.8)
+		(drill 0.4)
+		(layers "F.Cu" "B.Cu")
+		(net "GND")
+	)
+	(via
 		(at 133.181199 79.965979)
 		(size 0.8)
@@
 	)
 	(via
+		(at 129.17 51.23)
+		(size 0.8)
+		(drill 0.4)
+		(layers "F.Cu" "B.Cu")
+		(net "GND")
+	)
+	(via
 		(at 145.29 54.79)
 		(size 0.8)
@@
 	)
 	(via
+		(at 129.17 48.23)
+		(size 0.8)
+		(drill 0.4)
+		(layers "F.Cu" "B.Cu")
+		(net "GND")
+	)
+	(via
 		(at 148.37 47.97)
 		(size 0.8)
@@
 	)
 	(segment
-		(start 184.340001 70.269999)
-		(end 184.340001 68.669999)
+		(start 176.716239 63.433761)
+		(end 175.53 64.62)
 		(width 0.5)
 		(layer "F.Cu")
@@
 	)
 	(segment
-		(start 114.86027 63.5)
-		(end 117.9625 63.5)
+		(start 184.340001 70.269999)
+		(end 184.340001 68.669999)
 		(width 0.5)
 		(layer "F.Cu")
@@
 	)
 	(segment
-		(start 175.53 64.62)
-		(end 177.17 62.98)
+		(start 114.86027 63.5)
+		(end 117.9625 63.5)
 		(width 0.5)
 		(layer "F.Cu")
@@
 	)
 	(segment
+		(start 176.780691 63.433761)
+		(end 176.716239 63.433761)
+		(width 0.5)
+		(layer "F.Cu")
+		(net "+3V3")
+	)
+	(segment
 		(start 184.340001 84.900001)
 		(end 184.42 84.98)
@@
 	)
 	(segment
+		(start 175.53 64.62)
+		(end 175.36 64.62)
+		(width 0.5)
+		(layer "F.Cu")
+		(net "+3V3")
+	)
+	(segment
 		(start 181.87 94.386802)
 		(end 184.459017 91.797785)
@@
 	)
 	(segment
-		(start 175.36 64.62)
-		(end 175.53 64.62)
-		(width 0.5)
-		(layer "F.Cu")
-		(net "+3V3")
-	)
-	(segment
 		(start 143.42 123.48)
 		(end 143.42 120.73)
@@
 	)
 	(via
-		(at 177.17 62.98)
+		(at 176.780691 63.433761)
 		(size 0.8)
 		(drill 0.4)
@@
 	)
 	(segment
+		(start 176.780691 63.433761)
+		(end 177.623761 63.433761)
+		(width 0.5)
+		(layer "B.Cu")
+		(net "+3V3")
+	)
+	(segment
 		(start 184.42 84.98)
 		(end 184.67 85.23)
@@
 	)
 	(segment
-		(start 178.42 64.23)
-		(end 180.67 64.23)
-		(width 0.5)
+		(start 184.67 89.98)
+		(end 185.67 90.98)
+		(width 1)
 		(layer "B.Cu")
 		(net "+3V3")
 	)
 	(segment
-		(start 184.67 89.98)
-		(end 185.67 90.98)
-		(width 1)
+		(start 177.623761 63.433761)
+		(end 178.42 64.23)
+		(width 0.5)
 		(layer "B.Cu")
 		(net "+3V3")
@@
 	)
 	(segment
-		(start 177.17 62.98)
-		(end 178.42 64.23)
+		(start 178.42 64.23)
+		(end 180.67 64.23)
 		(width 0.5)
 		(layer "B.Cu")
