File: Hardware/PCB/LED_Coaster.kicad_sch (KiCad schematic)
At the start: 55 parts, among them J1 Input voltage, J2 Boot Option, J3 JTAG, J4 UART, SW1 SW_SPST, SW2 SW_DIP_x01, SW3 SW_DIP_x01, U1 ESP32-C3-WROOM-02-H4, U2 MCP1792x-3302xDB

Commit message: Latest and gratest PCB files from boa himself
Parts:
- removed D31, D32: LED, LED_SMD:LED_0805_2012Metric_Pad1.15x1.40mm_HandSolder, symbol Device:LED
- removed H2: MountingHole, MountingHole:MountingHole_4.3mm_M4_Pad_Via, symbol Mechanical:MountingHole
- removed J2: Boot Option, Connector_PinHeader_2.54mm:PinHeader_1x02_P2.54mm_Vertical, symbol Connector:Conn_01x02_Pin
- removed J3: JTAG, Connector_PinHeader_2.54mm:PinHeader_1x04_P2.54mm_Vertical, symbol Connector:Conn_01x04_Pin
- removed R7, R8: 150, Resistor_SMD:R_0805_2012Metric_Pad1.20x1.40mm_HandSolder, symbol Device:R
- removed SW2, SW3: SW_DIP_x01, Button_Switch_SMD:SW_SPDT_PCM12, symbol Switch:SW_DIP_x01
- removed U2: MCP1792x-3302xDB, Package_TO_SOT_SMD:SOT-223-3_TabPin2, symbol Regulator_Linear:MCP1792x-3302xDB
- added Btn1, Btn2: button, Button_Switch_SMD:SW_SPST_SKQG_WithStem, symbol Switch:SW_SPST
- added Btn3: Boot, Button_Switch_SMD:SW_SPST_SKQG_WithStem, symbol Switch:SW_SPST
- added C6, C7: 4.7uF, Capacitor_SMD:C_0805_2012Metric_Pad1.18x1.45mm_HandSolder, symbol Device:C_Small
- added D31, D32: SS34, Diode_SMD:D_SMA, symbol Diode:SS34
- added D33, D34: LED, LED_SMD:LED_0805_2012Metric_Pad1.15x1.40mm_HandSolder, symbol Device:LED
- added J3: USB_C_Receptacle_USB2.0_16P, Connector_USB:USB_C_Receptacle_HRO_TYPE-C-31-M-12, symbol Connector:USB_C_Receptacle_USB2.0_16P
- added R10, R11: 22, Resistor_SMD:R_0805_2012Metric_Pad1.20x1.40mm_HandSolder, symbol Device:R_Small
- added R12, R5, R8, R9: 1k, Resistor_SMD:R_0805_2012Metric_Pad1.20x1.40mm_HandSolder, symbol Device:R_Small
- added R2: 2k, Resistor_SMD:R_0805_2012Metric_Pad1.20x1.40mm_HandSolder, symbol Device:R_Small
- added R6, R7: 5.1K, Resistor_SMD:R_0805_2012Metric_Pad1.20x1.40mm_HandSolder, symbol Device:R_Small
- added SW1: SW_SPDT, Button_Switch_SMD:SW_SPDT_CK_JS102011SAQN, symbol Switch:SW_SPDT
- added U3: MCP73831-2-OT, Package_TO_SOT_SMD:SOT-23-5, symbol Battery_Management:MCP73831-2-OT
- added U4: AMS1117-3.3, Package_TO_SOT_SMD:SOT-223-3_TabPin2, symbol Regulator_Linear:AMS1117-3.3
- Btn4: renamed from SW1; value SW_SPST -> Enable; MPN (none) -> C318884
- C1: MPN (none) -> C15850
- C2: MPN (none) -> C28233
- C3: MPN (none) -> C28323
- C4, C5: MPN (none) -> C377773
- D1, D10, D11, D12, D13, D14, D15, D16, D17, D18, D19, D2, D20, D21, D22, D23, D24, D25, D26, D27, D28, D29, D3, D30, D4, D5, D6, D7, D8, D9: footprint LED_SMD:LED_WS2812B_PLCC4_5.0x5.0mm_P3.2mm -> Library:LED_WS2812_5050_handsolder; now not fitted
- H1, H3, H4, J4, U1: now not fitted
- J1: value Input voltage -> Li-po; footprint Connector_PinHeader_2.54mm:PinHeader_1x02_P2.54mm_Vertical -> Connector_JST:JST_EH_S2B-EH_1x02_P2.50mm_Horizontal; now not fitted
- R1, R3, R4: MPN (none) -> C17414
Connections:
- net +3V3: now also R8.1, R9.1, U4.2 (VO)
- net +5V: now also C6.2, D32.2 (A), D33.2 (A), J3.A4 (VBUS), J3.A9 (VBUS), J3.B4 (VBUS), J3.B9 (VBUS), U3.4 (V_{DD}); no longer C4.2, J1.2 (Pin_2)
- net GND: now also Btn1.1 (A), Btn2.1 (A), Btn3.2 (B), C6.1, C7.1, J3.A1 (GND), J3.A12 (GND), J3.B1 (GND), J3.B12 (GND), J3.S1 (SHIELD), R12.2, R6.2, R7.2, U4.1 (GND)
- net at U1.6 (IO7): now also D34.2 (A)
- net +BATT: now reaches D21.1 (VDD), D22.1 (VDD), D23.1 (VDD), D24.1 (VDD), D25.1 (VDD), D26.1 (VDD), D27.1 (VDD), D28.1 (VDD), D29.1 (VDD), D30.1 (VDD)
- net +BATT: now also C4.2, D1.1 (VDD), D10.1 (VDD), D11.1 (VDD), D12.1 (VDD), D13.1 (VDD), D14.1 (VDD), D15.1 (VDD), D16.1 (VDD), D17.1 (VDD), D18.1 (VDD), D19.1 (VDD), D2.1 (VDD), D20.1 (VDD), D3.1 (VDD), D4.1 (VDD), D5.1 (VDD), D6.1 (VDD), D7.1 (VDD), D8.1 (VDD), D9.1 (VDD), SW1.3 (C), U4.3 (VI)
- net at U1.8 (IO9): now also Btn3.1 (A)
- net at U1.13 (IO18): now also R10.1
- net at U1.14 (IO19): now also R11.1
- net at U1.15 (IO3): now also Btn2.2 (B), R9.2
- net at U1.16 (IO2): now also Btn1.2 (B), R8.2
- new net: D33.1 (K), R5.1
- new net: D34.1 (K), R12.1
- new net: R5.2, U3.1 (STAT)
- new net: R2.2, U3.2 (V_{SS})
- new net: C7.2, D31.2 (A), J1.2 (Pin_2), U3.3 (V_{BAT})
- new net: R2.1, U3.5 (PROG)
- new net: J3.A5 (CC1), R6.1
- new net: J3.B5 (CC2), R7.1
- new net: D31.1 (K), D32.1 (K), SW1.2 (B)
- new net D+: J3.A6 (D+), J3.B6 (D+), R11.2
- new net D-: J3.A7 (D-), J3.B7 (D-), R10.2
- no-connect marks 3 -> 9
Other:
- note added: "LDO"
- note added: "Li-Po"
- note added: "Li-Po charger"
- note added: "ON/OFF"
- moved on the sheet: C4, C5
