File: Hardware/PCB/LED_Coaster.kicad_sch (KiCad schematic)
At the start: 88 parts, among them J1 Li-po, J3 USB_C_Receptacle_USB2.0_16P, J4 UART, Q1 AO3401A, SW1 SW_SPDT, U1 ESP32-C3-WROOM-02-H4, U3 MCP73871-2CC, U4 TLV75533PDBVR

Commit message: Machine-place the LED ring and ESP32 module (double-sided assembly)
D1-D30 and U1 were excluded from assembly two ways: (dnp yes) in the
schematic, and no MPN field. Both are now cleared so JLCPCB places them.

  D1-D30  WS2812B-B/T            C2761795
  U1      ESP32-C3-WROOM-02-H4   C2944070

C2761795 is Standard-assembly only (MSL 5a), which matches the move to
double-sided anyway since Economic is single-side only.

J1 and J4 stay hand-soldered - both through-hole, so not SMT-placeable.

ORDERING.md updated: assembly model, cost expectation, and a warning that
the custom WS2812B footprint has no Fabrication Toolkit rotation rule.

Co-Authored-By: Claude Opus 5 <noreply@anthropic.com>
Parts:
- D1, D10, D11, D12, D13, D14, D15, D16, D17, D18, D19, D2, D20, D21, D22, D23, D24, D25, D26, D27, D28, D29, D3, D30, D4, D5, D6, D7, D8, D9: MPN (none) -> C2761795; now fitted
- U1: MPN (none) -> C2944070; now fitted
Changed lines of the file:
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@@
 		(on_board yes)
 		(in_pos_files yes)
-		(dnp yes)
+		(dnp no)
 		(fields_autoplaced yes)
 		(property "Reference" "D30"
@@
 			)
 		)
-		(property "MPN" ""
+		(property "MPN" "C2761795"
 			(at 275.59 102.87 0)
 			(hide yes)
@@
 		(on_board yes)
 		(in_pos_files yes)
-		(dnp yes)
+		(dnp no)
 		(fields_autoplaced yes)
 		(property "Reference" "D21"
@@
 			)
 		)
-		(property "MPN" ""
+		(property "MPN" "C2761795"
 			(at 69.85 102.87 0)
 			(hide yes)
@@
 		(on_board yes)
 		(in_pos_files yes)
-		(dnp yes)
+		(dnp no)
 		(fields_autoplaced yes)
 		(property "Reference" "D7"
@@
 			)
 		)
-		(property "MPN" ""
+		(property "MPN" "C2761795"
 			(at 208.28 58.42 0)
 			(hide yes)
@@
 		(on_board yes)
 		(in_pos_files yes)
-		(dnp yes)
+		(dnp no)
 		(fields_autoplaced yes)
 		(property "Reference" "D17"
@@
 			)
 		)
-		(property "MPN" ""
+		(property "MPN" "C2761795"
 			(at 436.88 58.42 0)
 			(hide yes)
@@
 		(on_board yes)
 		(in_pos_files yes)
-		(dnp yes)
+		(dnp no)
 		(fields_autoplaced yes)
 		(property "Reference" "D14"
@@
 			)
 		)
-		(property "MPN" ""
+		(property "MPN" "C2761795"
 			(at 368.3 58.42 0)
 			(hide yes)
@@
 		(on_board yes)
 		(in_pos_files yes)
-		(dnp yes)
+		(dnp no)
 		(fields_autoplaced yes)
 		(property "Reference" "D9"
@@
 			)
 		)
-		(property "MPN" ""
+		(property "MPN" "C2761795"
 			(at 254 58.42 0)
 			(hide yes)
@@
 		(on_board yes)
 		(in_pos_files yes)
-		(dnp yes)
+		(dnp no)
 		(fields_autoplaced yes)
 		(property "Reference" "D18"
@@
 			)
 		)
-		(property "MPN" ""
+		(property "MPN" "C2761795"
 			(at 459.74 58.42 0)
 			(hide yes)
@@
 		(on_board yes)
 		(in_pos_files yes)
-		(dnp yes)
+		(dnp no)
 		(fields_autoplaced yes)
 		(property "Reference" "D29"
@@
 			)
 		)
-		(property "MPN" ""
+		(property "MPN" "C2761795"
 			(at 252.73 102.87 0)
 			(hide yes)
@@
 		(on_board yes)
 		(in_pos_files yes)
-		(dnp yes)
+		(dnp no)
 		(fields_autoplaced yes)
 		(property "Reference" "D16"
@@
 			)
 		)
-		(property "MPN" ""
+		(property "MPN" "C2761795"
 			(at 414.02 58.42 0)
 			(hide yes)
@@
 		(on_board yes)
 		(in_pos_files yes)
-		(dnp yes)
+		(dnp no)
 		(fields_autoplaced yes)
 		(property "Reference" "D27"
@@
 			)
 		)
-		(property "MPN" ""
+		(property "MPN" "C2761795"
 			(at 207.01 102.87 0)
 			(hide yes)
@@
 		(on_board yes)
 		(in_pos_files yes)
-		(dnp yes)
+		(dnp no)
 		(fields_autoplaced yes)
 		(property "Reference" "D10"
@@
 			)
 		)
-		(property "MPN" ""
+		(property "MPN" "C2761795"
 			(at 276.86 58.42 0)
 			(hide yes)
@@
 		(on_board yes)
 		(in_pos_files yes)
-		(dnp yes)
+		(dnp no)
 		(fields_autoplaced yes)
 		(property "Reference" "D24"
@@
 			)
 		)
-		(property "MPN" ""
+		(property "MPN" "C2761795"
 			(at 138.43 102.87 0)
 			(hide yes)
@@
 		(on_board yes)
 		(in_pos_files yes)
-		(dnp yes)
+		(dnp no)
 		(fields_autoplaced yes)
 		(property "Reference" "D1"
@@
 			)
 		)
-		(property "MPN" ""
+		(property "MPN" "C2761795"
 			(at 70.485 58.42 0)
 			(hide yes)
@@
 		(on_board yes)
 		(in_pos_files yes)
-		(dnp yes)
+		(dnp no)
 		(fields_autoplaced yes)
 		(property "Reference" "D13"
@@
 			)
 		)
-		(property "MPN" ""
+		(property "MPN" "C2761795"
 			(at 345.44 58.42 0)
 			(hide yes)
@@
 		(on_board yes)
 		(in_pos_files yes)
-		(dnp yes)
+		(dnp no)
 		(fields_autoplaced yes)
 		(property "Reference" "D25"
@@
 			)
 		)
-		(property "MPN" ""
+		(property "MPN" "C2761795"
 			(at 161.29 102.87 0)
 			(hide yes)
@@
 		(on_board yes)
 		(in_pos_files yes)
-		(dnp yes)
+		(dnp no)
 		(fields_autoplaced yes)
 		(property "Reference" "D6"
@@
 			)
 		)
-		(property "MPN" ""
+		(property "MPN" "C2761795"
 			(at 185.42 58.42 0)
 			(hide yes)
@@
 		(on_board yes)
 		(in_pos_files yes)
-		(dnp yes)
+		(dnp no)
 		(fields_autoplaced yes)
 		(property "Reference" "D12"
@@
 			)
 		)
-		(property "MPN" ""
+		(property "MPN" "C2761795"
 			(at 322.58 58.42 0)
 			(hide yes)
@@
 		(on_board yes)
 		(in_pos_files yes)
-		(dnp yes)
+		(dnp no)
 		(fields_autoplaced yes)
 		(property "Reference" "D23"
@@
 			)
 		)
-		(property "MPN" ""
+		(property "MPN" "C2761795"
 			(at 115.57 102.87 0)
 			(hide yes)
@@
 		(on_board yes)
 		(in_pos_files yes)
-		(dnp yes)
+		(dnp no)
 		(fields_autoplaced yes)
 		(property "Reference" "D8"
@@
 			)
 		)
-		(property "MPN" ""
+		(property "MPN" "C2761795"
 			(at 231.14 58.42 0)
 			(hide yes)
@@
 		(on_board yes)
 		(in_pos_files yes)
-		(dnp yes)
+		(dnp no)
 		(fields_autoplaced yes)
 		(property "Reference" "D15"
@@
 			)
 		)
-		(property "MPN" ""
+		(property "MPN" "C2761795"
 			(at 391.16 58.42 0)
 			(hide yes)
@@
 		(on_board yes)
 		(in_pos_files yes)
-		(dnp yes)
+		(dnp no)
 		(fields_autoplaced yes)
 		(property "Reference" "D5"
@@
 			)
 		)
-		(property "MPN" ""
+		(property "MPN" "C2761795"
 			(at 162.56 58.42 0)
 			(hide yes)
@@
 		(on_board yes)
 		(in_pos_files yes)
-		(dnp yes)
+		(dnp no)
 		(property "Reference" "D2"
 			(at 104.775 54.7721 0)
@@
 			)
 		)
-		(property "MPN" ""
+		(property "MPN" "C2761795"
 			(at 93.98 58.42 0)
 			(hide yes)
@@
 		(on_board yes)
 		(in_pos_files yes)
-		(dnp yes)
+		(dnp no)
 		(fields_autoplaced yes)
 		(property "Reference" "U1"
@@
 			)
 		)
-		(property "MPN" ""
+		(property "MPN" "C2944070"
 			(at 158.75 190.5 0)
 			(hide yes)
@@
 		(on_board yes)
 		(in_pos_files yes)
-		(dnp yes)
+		(dnp no)
 		(fields_autoplaced yes)
 		(property "Reference" "D20"
@@
 			)
 		)
-		(property "MPN" ""
+		(property "MPN" "C2761795"
 			(at 505.46 58.42 0)
 			(hide yes)
@@
 		(on_board yes)
 		(in_pos_files yes)
-		(dnp yes)
+		(dnp no)
 		(property "Reference" "D3"
 			(at 127.635 54.7721 0)
@@
 			)
 		)
-		(property "MPN" ""
+		(property "MPN" "C2761795"
 			(at 116.84 58.42 0)
 			(hide yes)
@@
 		(on_board yes)
 		(in_pos_files yes)
-		(dnp yes)
+		(dnp no)
 		(fields_autoplaced yes)
 		(property "Reference" "D26"
@@
 			)
 		)
-		(property "MPN" ""
+		(property "MPN" "C2761795"
 			(at 184.15 102.87 0)
 			(hide yes)
@@
 		(on_board yes)
 		(in_pos_files yes)
-		(dnp yes)
+		(dnp no)
 		(property "Reference" "D4"
 			(at 150.495 54.7721 0)
@@
 			)
 		)
-		(property "MPN" ""
+		(property "MPN" "C2761795"
 			(at 139.7 58.42 0)
 			(hide yes)
@@
 		(on_board yes)
 		(in_pos_files yes)
-		(dnp yes)
+		(dnp no)
 		(fields_autoplaced yes)
 		(property "Reference" "D19"
@@
 			)
 		)
-		(property "MPN" ""
+		(property "MPN" "C2761795"
 			(at 482.6 58.42 0)
 			(hide yes)
@@
 		(on_board yes)
 		(in_pos_files yes)
-		(dnp yes)
+		(dnp no)
 		(fields_autoplaced yes)
 		(property "Reference" "D22"
@@
 			)
 		)
-		(property "MPN" ""
+		(property "MPN" "C2761795"
 			(at 92.71 102.87 0)
 			(hide yes)
@@
 		(on_board yes)
 		(in_pos_files yes)
-		(dnp yes)
+		(dnp no)
 		(fields_autoplaced yes)
 		(property "Reference" "D28"
@@
 			)
 		)
-		(property "MPN" ""
+		(property "MPN" "C2761795"
 			(at 229.87 102.87 0)
 			(hide yes)
@@
 		(on_board yes)
 		(in_pos_files yes)
-		(dnp yes)
+		(dnp no)
 		(fields_autoplaced yes)
 		(property "Reference" "D11"
@@
 			)
 		)
-		(property "MPN" ""
+		(property "MPN" "C2761795"
 			(at 299.72 58.42 0)
 			(hide yes)

Commit message: Mark J1 DNP, and correct what the guide says about exclusions
J1 is the through-hole JST battery connector, hand-soldered by
decision, and the guide has always listed it that way - but it was
never actually DNP. It came out of the Fabrication Toolkit as a
bom.csv line with an empty LCSC Part #: in the assembly list, and
unsourceable. Setting it DNP brings the count to 83 parts, 51 front
and 32 back, which is the number the guide already claimed.

Set in both places, because they do different jobs: the schematic
symbol carries (dnp yes) and the footprint carries (attr through_hole
dnp). The schematic is the one that matters - Update PCB from
Schematic overwrites a board-only change and puts the part quietly
back in the BOM.

The guide's account of how exclusion works was wrong, and this is
what it cost. It claimed a missing MPN would also keep a part out, and
that such a part "vanishes silently rather than appearing as a blank
line". J1 had no MPN, was not DNP, and produced exactly that blank
line. The toolkit filters on its EXCLUDE DNP option and nothing else.
The phase 7 BOM check now tells you to look for both failure modes.

Also corrects the board facts table, which still described the
pre-rework board at 46 front / 21 back. It is 51 / 33 physically, and
the revert-to-single-sided note now names the 33 back-side parts
instead of pointing at D1-D30 and U1 alone.

Co-Authored-By: Claude Opus 5 <noreply@anthropic.com>
Parts:
- J1: now not fitted
Changed lines of the file:
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@@
 		(on_board yes)
 		(in_pos_files yes)
-		(dnp no)
+		(dnp yes)
 		(property "Reference" "J1"
 			(at 462.28 256.54 0)

Commit message: Drop the buttons from assembly and re-source C20
JLCPCB had C318884 out of stock for BTN1-BTN4 and short on C296305
for C20.

The buttons are now DNP. The firmware reads none of them - there is
no pinMode or digitalRead anywhere in src/ - and BTN3 and BTN4 are the
ESP32 boot and reset buttons, which native USB-Serial-JTAG flashing
does not need. Hand-soldering four tactile switches later is easier
than finding a substitute that matches the land pattern, which needs
two 1.80 x 1.10 mm pads plus two mechanical in an 8.6 x 9.3 mm
envelope.

C20 moves from C296305 to C380336, a 10 V 22uF X5R 0805. The 6.3 V
alternative was cheaper but a 22uF X5R in an 0805 case loses most of
its capacitance under bias - at the 4.2 V this rail sits at, the 10 V
part holds roughly twice as much. It is a bulk reservoir on +LED_PWR,
so what matters is the capacitance that survives derating.

Both changes set in the schematic and the board, since Update PCB from
Schematic would otherwise put the parts back.

Assembly is now 79 parts, 47 front and 32 back. bom.csv is 23 lines
covering those 79, no line has an empty LCSC Part #, BOM and CPL name
the same designators, and nothing DNP appears in either.

Co-Authored-By: Claude Opus 5 <noreply@anthropic.com>
Parts:
- Btn1, Btn2, Btn3, Btn4: now not fitted
- C20: MPN C296305 -> C380336
Changed lines of the file:
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@@
 		(on_board yes)
 		(in_pos_files yes)
-		(dnp no)
+		(dnp yes)
 		(fields_autoplaced yes)
 		(property "Reference" "Btn3"
@@
 		(on_board yes)
 		(in_pos_files yes)
-		(dnp no)
+		(dnp yes)
 		(fields_autoplaced yes)
 		(property "Reference" "Btn1"
@@
 			)
 		)
-		(property "MPN" "C296305"
+		(property "MPN" "C380336"
 			(at 500.38 209.55 0)
 			(hide yes)
@@
 		(on_board yes)
 		(in_pos_files yes)
-		(dnp no)
+		(dnp yes)
 		(fields_autoplaced yes)
 		(property "Reference" "Btn2"
@@
 		(on_board yes)
 		(in_pos_files yes)
-		(dnp no)
+		(dnp yes)
 		(fields_autoplaced yes)
 		(property "Reference" "Btn4"

Commit message: Route charger status to the ESP32 and move the order to Economic
The board reports charge state in firmware now instead of on LEDs. U3's
three open-drain status outputs go to spare ESP32 pins - STAT1/LBO to
IO5, STAT2 to IO6, PG to IO10 - and the status LEDs D33/D35 with their
resistors R5/R16 are deleted.

Deleting them is required, not cosmetic: they pulled STAT1/STAT2 up to
+5V, and the ESP32-C3 is rated 3.6 V max on a pin. PG is what makes the
state decodable at all - per the MCP73871 Table 5-1, charging and low
battery share the same STAT1/STAT2 pair and differ only in PG.

The assembly model changes with it. The order is now Economic, single
sided, front only: 20 BOM lines and 47 placed parts for about $88,
against the $172.46 Standard double-sided quoted. Standard bills the
feeder fee on every line including Basic ones; Economic bills it only on
extended parts. The 28 back-side parts are the outer ring and its
decoupling, hand-soldered in a second stage, leaving J1 as the only part
stage one needs.

D1-D30 move to C55109525 (WS2812B-V7). C2761795 is Standard-only and one
such line forces the whole order off Economic. The V7 keeps the classic
1=VDD 2=DOUT 3=GND 4=DIN pinout so it drops in at 0 degrees; an SK6812
is also Economic-eligible but is 1=GND 2=DIN 3=VDD 4=DOUT, which at 0
degrees reverses the supply and destroys every LED.

C1, C3 and C5 merge onto the 4.7uF line - they were 25 V and 50 V parts
on a 3.3 V rail at twice the price of the 4.7uF already in the BOM.

Routing the three status nets through the B.Cu annulus split the ground
pour; two 1.0 mm bridges reconnect U3's ground island and C7.

Co-Authored-By: Claude Opus 5 <noreply@anthropic.com>
Parts:
- removed D33, D35: LED, LED_SMD:LED_0805_2012Metric_Pad1.15x1.40mm_HandSolder, symbol Device:LED
- removed R16, R5: 1k, Resistor_SMD:R_0805_2012Metric_Pad1.20x1.40mm_HandSolder, symbol Device:R_Small
- C1: value 10uF -> 4.7uF; MPN C15850 -> C1779
- C10, C11, C12, C13, C14, C15, C8, C9: now not fitted
- C3: value 1uF -> 4.7uF; MPN C28323 -> C1779
- C5: value 2.2uF -> 4.7uF; MPN C377773 -> C1779
- D1, D10, D11, D12, D13, D14, D15, D16, D17, D18, D19, D2, D20, D3, D4, D5, D6, D7, D8, D9: MPN C2761795 -> C55109525; now not fitted
- D21, D22, D23, D24, D25, D26, D27, D28, D29, D30: MPN C2761795 -> C55109525
Connections:
- net PG: now reaches U3.6 (~{PG})
- net PG: now also U1.10 (IO10)
- net STAT2: now reaches U3.7 (STAT2)
- net STAT2: now also U1.5 (IO6)
- net STAT1: now reaches U3.8 (STAT1/~{LBO})
- net STAT1: now also U1.4 (IO5)
- no-connect marks 9 -> 5

Commit message: Switch the LEDs to C26167850 and give the back-side parts thermal relief
Every WS2812B is MSL 5a and rated 240 C peak reflow. Economic PCBA runs a
255 C profile and does not bake, so JLCPCB rejects them at cart time no
matter what the part page's PCBA Type field claims - that field is
catalogue metadata, not what the ordering system enforces. C55109525,
C5380881 and both house-brand parts all advertise "Economic and Standard"
and all fail. Only the cart is authoritative.

TUOZHAN TZ-5050S2RGB-5V-I4-H1 clears it: MSL 3, 250 C peak, qualified at
260 C x 10 s twice with 0/22 failures. Verified accepted as Economic.

It is a better part here besides. Classic 1=VDD 2=DOU 3=GND 4=DIN pinout
so it drops in at 0 degrees; 80 us reset instead of 280, which retires the
delay(1) contingency the V7 would have needed; GRB order and bit timing
that FastLED's WS2812 driver already sits inside, so no firmware change at
all. 12 mA/channel against ~18-20 takes full white from ~1.8 A to ~1.08 A,
which largely retires the MCP73871 1 A system-load concern, and it is
brighter on green and blue despite the lower current.

D1-D20 and C8-C15 now carry zone_connect 1. The GND pour is solid, and the
datasheet allows an iron at 315 C for under 3 seconds once only - those
fight each other on a pad tied straight into a plane. Thermal relief on
just the hand-soldered back-side parts leaves the machine-assembled front
reflowing as before and keeps U3's exposed pad solid, as it needs to be.

Ordered: 20 lines, 47 parts, 7 extended. $83.36 PCBA plus $2.00 for the
boards against the $172.46 the first Standard double-sided quote came to.

Co-Authored-By: Claude Opus 5 <noreply@anthropic.com>
Parts:
- D1, D10, D11, D12, D13, D14, D15, D16, D17, D18, D19, D2, D20, D21, D22, D23, D24, D25, D26, D27, D28, D29, D3, D30, D4, D5, D6, D7, D8, D9: MPN C55109525 -> C26167850
Changed lines of the file:
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@@
 			)
 		)
-		(property "MPN" "C55109525"
+		(property "MPN" "C26167850"
 			(at 275.59 102.87 0)
 			(hide yes)
@@
 			)
 		)
-		(property "MPN" "C55109525"
+		(property "MPN" "C26167850"
 			(at 69.85 102.87 0)
 			(hide yes)
@@
 			)
 		)
-		(property "MPN" "C55109525"
+		(property "MPN" "C26167850"
 			(at 208.28 58.42 0)
 			(hide yes)
@@
 			)
 		)
-		(property "MPN" "C55109525"
+		(property "MPN" "C26167850"
 			(at 436.88 58.42 0)
 			(hide yes)
@@
 			)
 		)
-		(property "MPN" "C55109525"
+		(property "MPN" "C26167850"
 			(at 368.3 58.42 0)
 			(hide yes)
@@
 			)
 		)
-		(property "MPN" "C55109525"
+		(property "MPN" "C26167850"
 			(at 254 58.42 0)
 			(hide yes)
@@
 			)
 		)
-		(property "MPN" "C55109525"
+		(property "MPN" "C26167850"
 			(at 459.74 58.42 0)
 			(hide yes)
@@
 			)
 		)
-		(property "MPN" "C55109525"
+		(property "MPN" "C26167850"
 			(at 252.73 102.87 0)
 			(hide yes)
@@
 			)
 		)
-		(property "MPN" "C55109525"
+		(property "MPN" "C26167850"
 			(at 414.02 58.42 0)
 			(hide yes)
@@
 			)
 		)
-		(property "MPN" "C55109525"
+		(property "MPN" "C26167850"
 			(at 207.01 102.87 0)
 			(hide yes)
@@
 			)
 		)
-		(property "MPN" "C55109525"
+		(property "MPN" "C26167850"
 			(at 276.86 58.42 0)
 			(hide yes)
@@
 			)
 		)
-		(property "MPN" "C55109525"
+		(property "MPN" "C26167850"
 			(at 138.43 102.87 0)
 			(hide yes)
@@
 			)
 		)
-		(property "MPN" "C55109525"
+		(property "MPN" "C26167850"
 			(at 70.485 58.42 0)
 			(hide yes)
@@
 			)
 		)
-		(property "MPN" "C55109525"
+		(property "MPN" "C26167850"
 			(at 345.44 58.42 0)
 			(hide yes)
@@
 			)
 		)
-		(property "MPN" "C55109525"
+		(property "MPN" "C26167850"
 			(at 161.29 102.87 0)
 			(hide yes)
@@
 			)
 		)
-		(property "MPN" "C55109525"
+		(property "MPN" "C26167850"
 			(at 185.42 58.42 0)
 			(hide yes)
@@
 			)
 		)
-		(property "MPN" "C55109525"
+		(property "MPN" "C26167850"
 			(at 322.58 58.42 0)
 			(hide yes)
@@
 			)
 		)
-		(property "MPN" "C55109525"
+		(property "MPN" "C26167850"
 			(at 115.57 102.87 0)
 			(hide yes)
@@
 			)
 		)
-		(property "MPN" "C55109525"
+		(property "MPN" "C26167850"
 			(at 231.14 58.42 0)
 			(hide yes)
@@
 			)
 		)
-		(property "MPN" "C55109525"
+		(property "MPN" "C26167850"
 			(at 391.16 58.42 0)
 			(hide yes)
@@
 			)
 		)
-		(property "MPN" "C55109525"
+		(property "MPN" "C26167850"
 			(at 162.56 58.42 0)
 			(hide yes)
@@
 			)
 		)
-		(property "MPN" "C55109525"
+		(property "MPN" "C26167850"
 			(at 93.98 58.42 0)
 			(hide yes)
@@
 			)
 		)
-		(property "MPN" "C55109525"
+		(property "MPN" "C26167850"
 			(at 505.46 58.42 0)
 			(hide yes)
@@
 			)
 		)
-		(property "MPN" "C55109525"
+		(property "MPN" "C26167850"
 			(at 116.84 58.42 0)
 			(hide yes)
@@
 			)
 		)
-		(property "MPN" "C55109525"
+		(property "MPN" "C26167850"
 			(at 184.15 102.87 0)
 			(hide yes)
@@
 			)
 		)
-		(property "MPN" "C55109525"
+		(property "MPN" "C26167850"
 			(at 139.7 58.42 0)
 			(hide yes)
@@
 			)
 		)
-		(property "MPN" "C55109525"
+		(property "MPN" "C26167850"
 			(at 482.6 58.42 0)
 			(hide yes)
@@
 			)
 		)
-		(property "MPN" "C55109525"
+		(property "MPN" "C26167850"
 			(at 92.71 102.87 0)
 			(hide yes)
@@
 			)
 		)
-		(property "MPN" "C55109525"
+		(property "MPN" "C26167850"
 			(at 229.87 102.87 0)
 			(hide yes)
@@
 			)
 		)
-		(property "MPN" "C55109525"
+		(property "MPN" "C26167850"
 			(at 299.72 58.42 0)
 			(hide yes)
